File: ece137b_lab.kicad_sch (KiCad schematic)
At the start: 0 parts

Commit message: hahaha
Parts:
- added C1: 0.56u, Capacitor_THT:C_Rect_L10.0mm_W4.0mm_P7.50mm_FKS3_FKP3, symbol Device:C
- added C10: 470pF, Capacitor_THT:C_Radial_D6.3mm_H5.0mm_P2.50mm, symbol Device:C
- added C2, C3: C, Capacitor_THT:C_Radial_D6.3mm_H5.0mm_P2.50mm, symbol Device:C
- added C4, C5: 1n, Capacitor_THT:C_Radial_D6.3mm_H5.0mm_P2.50mm, symbol Device:C
- added C6, C8: 0.1u, Capacitor_THT:C_Radial_D6.3mm_H5.0mm_P2.50mm, symbol Device:C
- added C7, C9: 1u, Capacitor_THT:C_Radial_D6.3mm_H5.0mm_P2.50mm, symbol Device:C
- added J1, J2, J3: 575-8, 137b:CONN_575-8_KEY, symbol 137b:575-8
- added J4, J5, J6, J7: 132134, 137b:AMPHENOL_132134, symbol 137b:132134
- added JP1, JP2, JP7, JP8: SolderJumper_2_Open, Jumper:SolderJumper-2_P1.3mm_Open_Pad1.0x1.5mm, symbol Jumper:SolderJumper_2_Open
- added L1: 51u, 137b:CTX50-1-52-R, symbol Device:L
- added Q10: 2N3906, Package_TO_SOT_THT:TO-92_Inline, symbol Transistor_BJT:2N3906
- added Q11, Q13: BSS138, Package_TO_SOT_SMD:SOT-23, symbol Transistor_FET:BSS138
- added Q14, Q15: BSS84, Package_TO_SOT_SMD:SOT-23, symbol Transistor_FET:BSS84
- added Q5, Q7: PMOS, 137b:TO-251-3_Vertical, symbol Simulation_SPICE:PMOS
- added Q6, Q8: NMOS, 137b:TO-251-3_Vertical, symbol Simulation_SPICE:NMOS
- added Q9: 2N3904, Package_TO_SOT_THT:TO-92_Inline, symbol Transistor_BJT:2N3904
- added R1: 60, Resistor_THT:R_Axial_DIN0207_L6.3mm_D2.5mm_P10.16mm_Horizontal, symbol Device:R
- added R10: 2k, Resistor_THT:R_Axial_DIN0207_L6.3mm_D2.5mm_P10.16mm_Horizontal, symbol Device:R
- added R11: 1.8k, Resistor_THT:R_Axial_DIN0207_L6.3mm_D2.5mm_P10.16mm_Horizontal, symbol Device:R
- added R12, R13: 5, Resistor_THT:R_Axial_DIN0207_L6.3mm_D2.5mm_P10.16mm_Horizontal, symbol Device:R
- added R14: 330, Resistor_THT:R_Axial_DIN0207_L6.3mm_D2.5mm_P10.16mm_Horizontal, symbol Device:R
- added R15: 250, Resistor_THT:R_Axial_DIN0207_L6.3mm_D2.5mm_P10.16mm_Horizontal, symbol Device:R
- added R16: 8, Resistor_THT:R_Axial_DIN0207_L6.3mm_D2.5mm_P10.16mm_Horizontal, symbol Device:R
- added R2: 150, Resistor_THT:R_Axial_DIN0207_L6.3mm_D2.5mm_P10.16mm_Horizontal, symbol Device:R
- added R3: 80, Resistor_THT:R_Axial_DIN0207_L6.3mm_D2.5mm_P10.16mm_Horizontal, symbol Device:R
- added R4: 50, Resistor_THT:R_Axial_DIN0207_L6.3mm_D2.5mm_P10.16mm_Horizontal, symbol Device:R
- added R5: 8, Package_TO_SOT_THT:TO-220-2_Vertical, symbol Device:R
- added R6, R7, R8, R9: R, Resistor_THT:R_Axial_DIN0207_L6.3mm_D2.5mm_P10.16mm_Horizontal, symbol Device:R
- added TP1, TP10, TP11, TP2, TP7, TP8, TP9: 5002, 137b:KEYSTONE_5002, symbol 137b:5002
- added U1: (no value), 137b:DIP-8_W7.62mm, symbol 137b:ad790
- added U10, U9: LM318N, 137b:N08E, symbol Amplifier_Operational:LM318N
- added U4: SE555P, Package_DIP:DIP-8_W7.62mm, symbol Timer:SE555P
Connections:
- new net: C2.1, JP2.2 (B), U9.6
- new net: C2.2, R6.1, U9.2 (-)
- new net: R7.2, TP9.TP, U10.6, U9.3 (+)
- new net: C10.1, Q10.2 (B), Q9.2 (B), R14.2
- new net: C10.2, JP7.1 (A), R14.1, TP8.TP
- new net: C3.2, R7.1
- new net: Q11.3 (D), Q13.1 (G), Q15.1 (G), R3.2
- new net: Q6.1 (D), Q8.2 (G), R4.2
- new net: Q13.3 (D), Q6.2 (G), R2.2
- new net: Q9.3 (C), R15.1
- new net: Q10.1 (E), Q9.1 (E), R16.1
- new net: J4.1, JP2.1 (A), TP2.TP, U1.3 (-)
- new net: C3.1, R8.1, R9.2, U10.2 (-)
- new net: JP8.1 (A), R8.2
- new net: C1.1, J6.1, L1.2, R5.1
- new net: C9.2, R12.2
- new net: Q14.1 (G), R16.2
- new net: C4.2, U4.5 (CONT)
- new net: C7.2, R13.2
- new net: J5.1, JP1.2 (B), TP1.TP, U1.2 (+)
- new net: Q5.1 (D), Q7.2 (G), R4.1
- new net: Q15.3 (D), Q5.2 (G), R2.1
- new net: JP7.2 (B), U1.7 (Q)
- new net: Q11.1 (G), Q14.3 (D), R1.1
- new net +10V: C6.2, J1.1, Q15.2 (S), Q5.3 (S), Q7.3 (S), R13.1, R3.1, U1.1 (V+), U10.7 (V+), U9.7 (V+)
- new net +2V5: R10.1, U4.4 (~{RST}), U4.8 (VCC)
- new net +5V: Q14.2 (S), R15.2, U1.5 (LATCH), U1.8 (V_logic)
- new net -10V: C8.2, J2.1, Q11.2 (S), Q13.2 (S), Q6.3 (S), Q8.3 (S), R1.2, R12.1, U1.4 (V-), U10.4 (V-), U9.4 (V-)
- new net -2V5: C4.1, C5.2, U4.1 (GND)
- new net 555_out: JP1.1 (A), TP10.TP, U4.3 (OUT)
- new net GND: C1.2, C6.1, C7.1, C8.1, C9.1, J3.1, J4.G1, J4.G2, J4.G3, J4.G4, J5.G1, J5.G2, J5.G3, J5.G4, J6.G1, J6.G2, J6.G3, J6.G4, J7.G1, J7.G2, J7.G3, J7.G4, Q10.3 (C), R5.2, R6.2, U1.6 (GND), U10.3 (+)
- new net V_in: J7.1, R9.1, TP7.TP
- new net V_sw: JP8.2 (B), L1.1, Q7.1 (D), Q8.1 (D), TP11.TP
- new net disch: R10.2, R11.1, U4.7 (DISCH)
- new net thres: C5.1, R11.2, U4.2 (TRIG), U4.6 (THRES)
Other:
- added sheet Regulators (Regulators.kicad_sch)
- note added: "555 Timer (Triangle Wave Generator)"
- note added: "Comparator"
- note added: "Driver"
- note added: "Feedback Network (Two Integrators, one has a zero for lead lag compensation)"
